Commit message: Mount manipulator arm on Go2

File: urdf/go2_unitree/urdf/go2_gz.urdf (robot description, URDF)
Before this commit: robot go2_description, 29 links, 28 joints
Links:
- added link arm_base, mass 0.15; collision mesh filename=package://champ_description/meshes/arm/base.stl scale=0.001 0.001 0.001; visual mesh filename=package://champ_description/meshes/arm/base.stl scale=0.001 0.001 0.001
- added link base_mount
- added link lower_arm, mass 0.1; collision mesh filename=package://champ_description/meshes/arm/lower_arm.stl scale=0.001 0.001 0.001; visual mesh filename=package://champ_description/meshes/arm/lower_arm.stl scale=0.001 0.001 0.001
- added link upper_arm, mass 0.1; collision mesh filename=package://champ_description/meshes/arm/upper_arm.stl scale=0.001 0.001 0.001; visual mesh filename=package://champ_description/meshes/arm/upper_arm.stl scale=0.001 0.001 0.001
- added link wrist1, mass 0.05; collision mesh filename=package://champ_description/meshes/arm/wrist1.stl scale=0.001 0.001 0.001; visual mesh filename=package://champ_description/meshes/arm/wrist1.stl scale=0.001 0.001 0.001
- added link wrist2, mass 0.05; collision mesh filename=package://champ_description/meshes/arm/wrist2.stl scale=0.001 0.001 0.001; visual mesh filename=package://champ_description/meshes/arm/wrist2.stl scale=0.001 0.001 0.001
Joints:
- added joint base_joint: type revolute, parent base_mount, child arm_base, origin xyz=0 0 0 rpy=0 0 0, axis 0 0 1, limit lower=-1.57079632679 upper=1.57079632679 effort=25 velocity=1.5
- added joint lower_arm_joint: type revolute, parent arm_base, child lower_arm, origin xyz=0 0 0.035 rpy=0 0 0, axis 0 1 0, limit lower=-1.57079632679 upper=1.57079632679 effort=25 velocity=1.5
- added joint robot_to_arm_joint: type fixed, parent base, child base_mount, origin xyz=0.08 0 0.057 rpy=0 0 0
- added joint upper_arm_joint: type revolute, parent lower_arm, child upper_arm, origin xyz=0.195 0 0 rpy=0 0 0, axis 0 1 0, limit lower=-1.57079632679 upper=1.57079632679 effort=25 velocity=1.5
- added joint wrist1_joint: type revolute, parent upper_arm, child wrist1, origin xyz=0.195 0 0 rpy=0 0 0, axis 0 1 0, limit lower=-1.57079632679 upper=1.57079632679 effort=25 velocity=1.5
- added joint wrist2_joint: type revolute, parent wrist1, child wrist2, origin xyz=0.065 0 0 rpy=0 0 0, axis 1 0 0, limit lower=-1.57079632679 upper=1.57079632679 effort=25 velocity=1.5

File: urdf/go2_unitree/urdf/go2_gz.urdf.xacro (robot description, xacro)
@@ -3,4 +3,11 @@
   <!-- Include base go2 URDF -->
   <xacro:include filename="$(find champ_description)/urdf/go2.urdf"/>
+  <!-- 5-DOF manipulator arm mounted on top of the body, forward of center
+       and above the base collision box (0.3762 x 0.0935 x 0.114, top face
+       at z=0.057) so it doesn't intersect the body mesh -->
+  <xacro:include filename="$(find champ_description)/urdf/arm.urdf.xacro"/>
+  <xacro:champ_arm parent="base">
+    <origin rpy="0 0 0" xyz="0.08 0 0.057"/>
+  </xacro:champ_arm>
   <!-- Gazebo Harmonic gz_ros2_control plugin -->
   <gazebo>
@@ -75,4 +82,29 @@
       <state_interface name="velocity"/>
     </joint>
+    <joint name="base_joint">
+      <command_interface name="position"/>
+      <state_interface name="position"><param name="initial_value">0.0</param></state_interface>
+      <state_interface name="velocity"/>
+    </joint>
+    <joint name="lower_arm_joint">
+      <command_interface name="position"/>
+      <state_interface name="position"><param name="initial_value">0.0</param></state_interface>
+      <state_interface name="velocity"/>
+    </joint>
+    <joint name="upper_arm_joint">
+      <command_interface name="position"/>
+      <state_interface name="position"><param name="initial_value">0.0</param></state_interface>
+      <state_interface name="velocity"/>
+    </joint>
+    <joint name="wrist1_joint">
+      <command_interface name="position"/>
+      <state_interface name="position"><param name="initial_value">0.0</param></state_interface>
+      <state_interface name="velocity"/>
+    </joint>
+    <joint name="wrist2_joint">
+      <command_interface name="position"/>
+      <state_interface name="position"><param name="initial_value">0.0</param></state_interface>
+      <state_interface name="velocity"/>
+    </joint>
   </ros2_control>
   <!-- IMU sensor on base -->

Commit message: Add base_footprint frame for RTAB-Map and enable grid ray tracing

File: urdf/go2_unitree/urdf/go2_gz.urdf (robot description, URDF)
Before this commit: robot go2_description, 38 links, 37 joints
Links:
- added link base_footprint
Joints:
- added joint base_footprint_joint: type fixed, parent base, child base_footprint, origin xyz=0 0 -0.22 rpy=0 0 0

File: urdf/go2_unitree/urdf/go2_gz.urdf.xacro (robot description, xacro)
@@ -26,5 +26,5 @@
        unconditionally every update, independent of ros2_control's
        controller_manager lifecycle. Launch files bridge this straight to
-       ROS /joint_states -- see launch/gazebo_go2.launch.py's bridge args. -->
+       ROS /joint_states, see launch/gazebo_go2.launch.py's bridge args. -->
   <gazebo>
     <plugin filename="libgz-sim-joint-state-publisher-system.so"
@@ -215,5 +215,5 @@
   <!-- Forward-facing RGB camera for the RViz picture-in-picture inset (see
        ros2/champ_navigation/rviz/slam.rviz's Image display). Native gz-sim
-       sensor, same style as the imu/lidar blocks above -- no gazebo_ros
+       sensor, same style as the imu/lidar blocks above, no gazebo_ros
        plugin (that's classic Gazebo only); bridge via ros_gz_bridge in
        launch/slam3d_go2.launch.py instead. -->
@@ -239,3 +239,17 @@
     </sensor>
   </gazebo>
+  <!-- Ground-projected frame for RTAB-Map (see slam3d_go2.launch.py's
+       frame_id). "base" sits at nominal_height=0.22m (config/go2_champ/
+       gait.yaml) above the ground, so using it directly as RTAB-Map's
+       frame_id would put the map/grid's z=0 origin at body height instead
+       of the ground, and the 2D occupancy grid then renders floating above
+       where the feet actually are. base_footprint is fixed (not measured
+       ride height) because SLAM needs a frame rigidly attached to the
+       robot, same fix as Magi's magi_slam (ali-pahlevani/Magi). -->
+  <link name="base_footprint"/>
+  <joint name="base_footprint_joint" type="fixed">
+    <parent link="base"/>
+    <child link="base_footprint"/>
+    <origin xyz="0 0 -0.22" rpy="0 0 0"/>
+  </joint>
 </robot>
